File: ldrd/ldrd.kicad_pcb (KiCad board)
At the start: 4 copper layers, 137.3 x 100 mm, 63 parts, among them J1 USB_C_Receptacle_USB2.0, J2 Conn_01x04, J3 Conn_01x04, Q1 UMH3N, SW1 Light Switch, SW2 Scroll Click Wheel, U1 SN74LV1T34DBV, U2 AP2114HA-3.3, U3 CH340C, U4 T-Micro32_Plus

Commit message: add lcd label
Other:
- board text added: "LCD"
Changed lines of the file:
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@@
       (drillshape 0)
       (scaleselection 1)
-      (outputdirectory "PCBway/")
+      (outputdirectory "drill/")
     )
   )
@@
     (effects (font (size 1.5 1.5) (thickness 0.3)))
   )
+  (gr_text "LCD" (at 144.78 81.28) (layer "F.SilkS")
+    (effects (font (size 1.5 1.5) (thickness 0.3)))
+  )
